Commit message: - Added IMU - Fixed gazebo controller errors - Changed Docker to run ROS1 noetic

File: ws/src/duckiebot_description/urdf/duckiebot.xacro (robot description, xacro)
@@ -1,231 +1,201 @@
-<?xml version='1.0'?>
+<?xml version="1.0"?>
 <robot name="duckiebot" xmlns:xacro="http://www.ros.org/wiki/xacro">
+  <!-- Properties -->
   <xacro:property name="cameraSize" value="0.01"/>
   <xacro:property name="cameraMass" value="0.01"/>
   <xacro:property name="compuMass" value="0.01"/>
-  <!-- Constants -->
   <xacro:property name="PI" value="3.1415926535897931"/>
-  <!-- Chassis properties -->
+  <!-- Chassis -->
   <xacro:property name="chassisHeight" value="0.0623"/>
   <xacro:property name="chassisLength" value="0.198"/>
   <xacro:property name="chassisWidth" value="0.119"/>
   <xacro:property name="chassisMass" value="0.15"/>
-  <!-- Caster wheel properties -->
+  <!-- Caster -->
   <xacro:property name="casterRadius" value="0.021"/>
   <xacro:property name="casterMass" value="0.09"/>
   <xacro:property name="casterOffsetX" value="0.091"/>
-  <!-- Differential-drive wheels properties -->
+  <!-- Wheels -->
   <xacro:property name="wheelWidth" value="0.026"/>
   <xacro:property name="wheelRadius" value="0.032"/>
   <xacro:property name="wheelMass" value="0.05"/>
   <xacro:property name="wheelOffsetY" value="0.037"/>
-  <xacro:include filename="$(find duckiebot_description)/urdf/duckiebot.gazebo" />
-  <xacro:include filename="$(find duckiebot_description)/urdf/materials.xacro" />
-  <xacro:include filename="$(find duckiebot_description)/urdf/macros.xacro" />
+  <!-- Gazebo Materials -->
+  <xacro:include filename="$(find duckiebot_description)/urdf/materials.xacro"/>
+  <xacro:include filename="$(find duckiebot_description)/urdf/macros.xacro"/>
+  <xacro:include filename="$(find duckiebot_description)/urdf/duckiebot.gazebo"/>
   <pose>0 0 0 0 0 0</pose>
-  <link name='chassis'>
+  <!-- ======================= CHASSIS ======================= -->
+  <link name="chassis">
     <inertial>
       <mass value="${chassisMass}"/>
-      <origin xyz="-0.05 0 0" rpy=" 0 0 0"/>
-      <inertia
-        ixx="1.56167e-05" ixy="0.0" ixz="0.0"
-        iyy="1.56167e-05" iyz="0.0"
-        izz="2.56e-05"/>
-    </inertial>
-    <collision name='collision'>
-      <origin xyz="0 0 0" rpy=" 0 0 0"/>
+      <origin xyz="-0.05 0 0"/>
+      <inertia ixx="1.56167e-05" ixy="0" ixz="0"
+               iyy="1.56167e-05" iyz="0"
+               izz="2.56e-05"/>
+    </inertial>
+    <visual>
+      <origin xyz="0 0 0"/>
       <geometry>
         <mesh filename="package://duckiebot_description/meshes/duckiebotFrame.dae"/>
       </geometry>
-    </collision>
-    <visual name='chassis_visual'>
-      <origin xyz="0 0 0" rpy=" 0 0 0"/>
+      <material name="red"/>
+    </visual>
+    <collision>
+      <origin xyz="0 0 0"/>
       <geometry>
         <mesh filename="package://duckiebot_description/meshes/duckiebotFrame.dae"/>
       </geometry>
-      <material name="red"/>
-    </visual>
-  </link>
+    </collision>
+  </link>
+  <!-- ======================= WHEELS ======================= -->
   <link name="left_wheel">
-    <origin xyz="0 0 0" rpy="0 0 0"/>
-    <collision name="collision">
-      <origin xyz="0 -0.07 0" rpy="0 0 0"/>
+    <inertial>
+      <mass value="${wheelMass}"/>
+      <origin xyz="0 0 0"/>
+      <inertia ixx="0.561e-05" iyy="0.561e-05" izz="1.56e-05" ixy="0" ixz="0" iyz="0"/>
+    </inertial>
+    <visual>
+      <origin xyz="0 -0.07 0"/>
       <geometry>
         <mesh filename="package://duckiebot_description/meshes/duckiebot_leftwheel.dae"/>
       </geometry>
-    </collision>
-    <visual name="left_wheel_visual">
-      <origin xyz="0 -0.07 0" rpy="0 0 0"/>
+      <material name="black"/>
+    </visual>
+    <collision>
+      <origin xyz="0 -0.07 0"/>
       <geometry>
         <mesh filename="package://duckiebot_description/meshes/duckiebot_leftwheel.dae"/>
       </geometry>
+    </collision>
+  </link>
+  <link name="right_wheel">
+    <inertial>
+      <mass value="${wheelMass}"/>
+      <origin xyz="0 0 0"/>
+      <inertia ixx="0.561e-05" iyy="0.561e-05" izz="1.56e-05" ixy="0" ixz="0" iyz="0"/>
+    </inertial>
+    <visual>
+      <origin xyz="0 0.07 0"/>
+      <geometry>
+        <mesh filename="package://duckiebot_description/meshes/duckiebot_rightwheel.dae"/>
+      </geometry>
       <material name="black"/>
     </visual>
-    <inertial>
-      <origin xyz="0 0 0" rpy="0 0 0"/>
-      <mass value="${wheelMass}"/>
-      <cylinder_inertia m="${wheelMass}" r="0.0325" h="0.02"/>
-      <inertia
-        ixx="0.56167e-05" ixy="0.0" ixz="0.0"
-        iyy="0.56167e-05" iyz="0.0"
-        izz="1.56e-05"/>
-    </inertial>
-  </link>
-  <link name="right_wheel">
-    <origin xyz="0 0 0" rpy="0 0 0"/>
-    <collision name="collision">
-      <origin xyz="0 0.07 0" rpy="0 0 0"/>
+    <collision>
+      <origin xyz="0 0.07 0"/>
       <geometry>
         <mesh filename="package://duckiebot_description/meshes/duckiebot_rightwheel.dae"/>
       </geometry>
     </collision>
-    <visual name="right_wheel_visual">
-      <origin xyz="0 0.07 0" rpy="0 0 0"/>
-      <geometry>
-        <mesh filename="package://duckiebot_description/meshes/duckiebot_rightwheel.dae"/>
-      </geometry>
-      <material name="black"/>
-    </visual>
-    <inertial>
-      <origin xyz="0 0 0" rpy="0 0 0"/>
-      <mass value="${wheelMass}"/>
-      <cylinder_inertia m="${wheelMass}" r="0.0325" h="0.01"/>
-      <inertia
-        ixx="0.56167e-05" ixy="0.0" ixz="0.0"
-        iyy="0.56167e-05" iyz="0.0"
-        izz="1.56e-05"/>
-    </inertial>
-  </link>
+  </link>
+  <!-- Wheel joints -->
   <joint type="continuous" name="left_wheel_hinge">
-    <origin xyz="0.0 0.07 0" rpy="0 0 0"/>
+    <parent link="chassis"/>
     <child link="left_wheel"/>
-    <parent link="chassis"/>
-    <axis xyz="0 1 0" rpy="0 0 0"/>
-    <limit effort="100" velocity="100"/>
-    <joint_properties damping="0.0" friction="0.0"/>
+    <origin xyz="0 0.07 0"/>
+    <axis xyz="0 1 0"/>
   </joint>
   <joint type="continuous" name="right_wheel_hinge">
-    <origin xyz="0.0 -0.07 0" rpy="0 0 0"/>
+    <parent link="chassis"/>
     <child link="right_wheel"/>
-    <parent link="chassis"/>
-    <axis xyz="0 1 0" rpy="0 0 0"/>
-    <limit effort="100" velocity="100"/>
-    <joint_properties damping="0.0" friction="0.0"/>
-  </joint>
-<!-- Computer -->
-<link name="computer">
-    <collision>
-      <origin xyz="0 0 0" rpy="0 0 0"/>
+    <origin xyz="0 -0.07 0"/>
+    <axis xyz="0 1 0"/>
+  </joint>
+  <!-- ======================= COMPUTER ======================= -->
+  <link name="computer">
+    <inertial>
+      <mass value="${compuMass}"/>
+      <origin xyz="0 0 0"/>
+      <inertia ixx="1e-6" iyy="1e-6" izz="1e-6"/>
+    </inertial>
+    <visual>
       <geometry>
         <mesh filename="package://duckiebot_description/meshes/duckiebot_computer.dae"/>
       </geometry>
-    </collision>
-    <visual name='comp_visual'>
-      <origin xyz="0 0 0" rpy=" 0 0 0"/>
+      <material name="blue"/>
+    </visual>
+    <collision>
       <geometry>
         <mesh filename="package://duckiebot_description/meshes/duckiebot_computer.dae"/>
       </geometry>
+    </collision>
+  </link>
+  <joint name="computer_joint" type="fixed">
+    <parent link="chassis"/>
+    <child link="computer"/>
+  </joint>
+  <!-- ======================= IMU (FIXED + WORKING) ======================= -->
+  <link name="imu_link">
+    <inertial>
+      <mass value="0.01"/>
+      <origin xyz="0 0 0"/>
+      <inertia ixx="1e-6" iyy="1e-6" izz="1e-6"/>
+    </inertial>
+    <visual>
+      <geometry>
+        <box size="0.01 0.01 0.01"/>
+      </geometry>
       <material name="blue"/>
     </visual>
-    <inertial>
-      <mass value="${compuMass}" />
-      <origin xyz="0 0 0" rpy="0 0 0"/>
-      <inertia ixx="1e-6" ixy="0" ixz="0" iyy="1e-6" iyz="0" izz="1e-6" />
-    </inertial>
-  </link>
-<link name="imu_link">
-  <inertial>
-    <mass value="0.01"/>
-    <origin xyz="0 0 0" rpy="0 0 0"/>
-    <inertia ixx="1e-6" ixy="0" ixz="0" iyy="1e-6" iyz="0" izz="1e-6"/>
-  </inertial>
-  <visual>
-    <origin xyz="0 0 0"/>
-    <geometry>
-      <box size="0.01 0.01 0.01"/>
-    </geometry>
-    <material name="blue"/>
-  </visual>
-  <collision>
-    <origin xyz="0 0 0"/>
-    <geometry>
-      <box size="0.01 0.01 0.01"/>
-    </geometry>
-  </collision>
-  <!-- Gazebo-native IMU -->
-  <gazebo>
+    <collision>
+      <geometry>
+        <box size="0.01 0.01 0.01"/>
+      </geometry>
+    </collision>
+  </link>
+  <joint name="imu_joint" type="fixed">
+    <parent link="computer"/>
+    <child link="imu_link"/>
+    <origin xyz="0 0 0.02"/>
+  </joint>
+  <gazebo reference="imu_link">
     <sensor type="imu" name="imu_sensor">
-      <always_on>1</always_on>
+      <always_on>true</always_on>
       <update_rate>50</update_rate>
-      <visualize>true</visualize>
-      <topic>imu/data_raw</topic>
+      <topicName>imu/data</topicName>
       <imu>
         <angular_velocity>
-          <x>1</x>
-          <y>1</y>
-          <z>1</z>
+          <x>1</x><y>1</y><z>1</z>
         </angular_velocity>
         <linear_acceleration>
-          <x>1</x>
-          <y>1</y>
-          <z>1</z>
+          <x>1</x><y>1</y><z>1</z>
         </linear_acceleration>
       </imu>
-      <noise>
-        <angular_velocity>
-          <mean>0.0</mean>
-          <stddev>0.0001</stddev>
-        </angular_velocity>
-        <linear_acceleration>
-          <mean>0.0</mean>
-          <stddev>0.0001</stddev>
-        </linear_acceleration>
-      </noise>
+      <plugin name="imu_plugin" filename="libgazebo_ros_imu_sensor.so">
+        <ros>
+          <namespace>/</namespace>
+        </ros>
+        <frameName>imu_link</frameName>
+      </plugin>
     </sensor>
   </gazebo>
-</link>
-<!-- Fixed joint attaching IMU to the computer -->
-<joint name="imu_joint" type="fixed">
-  <parent link="computer"/>
-  <child link="imu_link"/>
-  <origin xyz="0 0 0" rpy="0 0 0"/>
-</joint>
-  <joint name="computer_joint" type="fixed">
-    <axis xyz="0 0 0" />
-    <origin xyz="0 0 0" rpy="0 0 0"/>
-    <parent link="chassis"/>
-    <child link="computer"/>
-  </joint>
-<!-- Camera sensor -->
-<link name="camera">
-    <pose>0 0 0 0 0 0</pose>
-    <collision>
+  <!-- ======================= CAMERA ======================= -->
+  <link name="camera">
+    <inertial>
+      <mass value="${cameraMass}"/>
+      <origin xyz="0 0 0"/>
+      <inertia ixx="1e-6" iyy="1e-6" izz="1e-6"/>
+    </inertial>
+    <visual>
       <origin xyz="-0.05 0 -0.055" rpy="0 -0.1 0"/>
       <geometry>
         <mesh filename="package://duckiebot_description/meshes/duckiebot_camera.dae"/>
       </geometry>
-    </collision>
-    <visual name='camvisual'>
-      <origin xyz="-0.05 0 -0.055" rpy=" 0 -0.1 0"/>
+      <material name="black"/>
+    </visual>
+    <collision>
+      <origin xyz="-0.05 0 -0.055" rpy="0 -0.1 0"/>
       <geometry>
         <mesh filename="package://duckiebot_description/meshes/duckiebot_camera.dae"/>
       </geometry>
-      <material name="black"/>
-    </visual>
-    <inertial>
-      <mass value="${cameraMass}" />
-      <origin xyz="0 0 0" rpy="0 0 0"/>
-      <inertia ixx="1e-6" ixy="0" ixz="0" iyy="1e-6" iyz="0" izz="1e-6" />
-    </inertial>
-  </link>
-<!-- This joint info decides the pos of camera. Pitch(p in rpy) is angle to control orientation for duckiebot camera.After change values here, you need to change the pos info in collision part anf visual part just above.-->
+    </collision>
+  </link>
   <joint name="camera_joint" type="fixed">
-    <axis xyz="0 0 0" />
+    <parent link="chassis"/>
+    <child link="camera"/>
     <origin xyz="0.05 0 0.05" rpy="0 0.1 0"/>
-    <parent link="chassis"/>
-    <child link="camera"/>
   </joint>
 <!-- Transmissions for wheel joints -->
-  <transmission name="left_wheel_trans">
+  <!-- <transmission name="left_wheel_trans">
     <type>transmission_interface/SimpleTransmission</type>
     <joint name="left_wheel_hinge"/>
@@ -240,8 +210,8 @@
       <mechanicalReduction>1</mechanicalReduction>
     </actuator>
-  </transmission>
+  </transmission> -->
   <!-- Gazebo ROS Control plugin -->
-  <gazebo>
+  <!-- <gazebo>
     <plugin name="gazebo_ros_control" filename="libgazebo_ros_control.so"/>
-  </gazebo>
+  </gazebo> -->
 </robot>

Commit message: added robot state publisher to sim launch. static tf between frames. addedd joint_state_publisher to duckiebot.gazebo . fixed tf issues.

File: ws/src/duckiebot_description/urdf/duckiebot.xacro (robot description, xacro)
@@ -25,4 +25,20 @@
   <xacro:include filename="$(find duckiebot_gazebo)/urdf/duckiebot.gazebo"/>
   <pose>0 0 0 0 0 0</pose>
+  <!-- ======================= BASE_LINK (ROS Navigation Reference) ======================= -->
+  <link name="base_link">
+    <inertial>
+      <mass value="0.0"/>
+      <origin xyz="0 0 0"/>
+      <inertia ixx="0" ixy="0" ixz="0"
+              iyy="0" iyz="0"
+              izz="0"/>
+    </inertial>
+  </link>
+  <!-- Joint connecting base_link to chassis (raised by wheel radius) -->
+  <joint name="base_to_chassis" type="fixed">
+    <parent link="base_link"/>
+    <child link="chassis"/>
+    <origin xyz="0 0 ${wheelRadius}" rpy="0 0 0"/>
+  </joint>
   <!-- ======================= CHASSIS ======================= -->
   <link name="chassis">
@@ -107,5 +123,7 @@
       <mass value="${compuMass}"/>
       <origin xyz="0 0 0"/>
-      <inertia ixx="1e-6" iyy="1e-6" izz="1e-6"/>
+      <inertia ixx="1e-6" ixy="0" ixz="0"
+              iyy="1e-6" iyz="0"
+              izz="1e-6"/>
     </inertial>
     <visual>
@@ -130,5 +148,7 @@
       <mass value="0.01"/>
       <origin xyz="0 0 0"/>
-      <inertia ixx="1e-6" iyy="1e-6" izz="1e-6"/>
+      <inertia ixx="1e-6" ixy="0" ixz="0"
+              iyy="1e-6" iyz="0"
+              izz="1e-6"/>
     </inertial>
     <visual>
@@ -173,5 +193,7 @@
       <mass value="${cameraMass}"/>
       <origin xyz="0 0 0"/>
-      <inertia ixx="1e-6" iyy="1e-6" izz="1e-6"/>
+      <inertia ixx="1e-6" ixy="0" ixz="0"
+              iyy="1e-6" iyz="0"
+              izz="1e-6"/>
     </inertial>
     <visual>

Commit message: Increased IMU link mass, removed embedded robot from world file, and cleaned up plugins

File: ws/src/duckiebot_description/urdf/duckiebot.xacro (robot description, xacro)
@@ -173,14 +173,53 @@
     <sensor name="imu_sensor" type="imu">
       <always_on>true</always_on>
-      <update_rate>200</update_rate>
-      <visualize>true</visualize>
-      <topic>__default_topic__</topic>
-      <plugin filename="libgazebo_ros_imu_sensor.so" name="imu_plugin">
-        <topicName>imu_data</topicName>
-        <bodyName>imu_link</bodyName>
-        <updateRate>200.0</updateRate>
-        <gaussianNoise>0.0</gaussianNoise>
-        <xyzOffset>0 0 0</xyzOffset>
-        <rpyOffset>0 0 0</rpyOffset>
+      <imu>
+        <angular_velocity>
+          <x>
+            <noise type="gaussian">
+              <mean>0.0</mean>
+              <stddev>0.0</stddev>
+            </noise>
+          </x>
+          <y>
+            <noise type="gaussian">
+              <mean>0.0</mean>
+              <stddev>0.0</stddev>
+            </noise>
+          </y>
+          <z>
+            <noise type="gaussian">
+              <mean>0.0</mean>
+              <stddev>0.0</stddev>
+            </noise>
+          </z>
+        </angular_velocity>
+        <linear_acceleration>
+          <x>
+            <noise type="gaussian">
+              <mean>0.0</mean>
+              <stddev>0.0</stddev>
+            </noise>
+          </x>
+          <y>
+            <noise type="gaussian">
+              <mean>0.0</mean>
+              <stddev>0.0</stddev>
+            </noise>
+          </y>
+          <z>
+            <noise type="gaussian">
+              <mean>0.0</mean>
+              <stddev>0.0</stddev>
+            </noise>
+          </z>
+        </linear_acceleration>
+      </imu>
+      <plugin name="imu_plugin" filename="libgazebo_ros_imu_sensor.so">
+        <ros>
+          <namespace>duckiebot</namespace>
+        </ros>
+        <updateRateHZ>200</updateRateHZ>
+        <robotNamespace>duckiebot</robotNamespace>
+        <topicName>imu/data</topicName>
         <frameName>imu_link</frameName>
         <initialOrientationAsReference>false</initialOrientationAsReference>
@@ -216,22 +255,3 @@
     <origin xyz="0.05 0 0.05" rpy="0 0.1 0"/>
   </joint>
-<!-- Transmissions for wheel joints -->
-  <!-- <transmission name="left_wheel_trans">
-    <type>transmission_interface/SimpleTransmission</type>
-    <joint name="left_wheel_hinge"/>
-    <actuator name="left_wheel_motor">
-      <mechanicalReduction>1</mechanicalReduction>
-    </actuator>
-  </transmission>
-  <transmission name="right_wheel_trans">
-    <type>transmission_interface/SimpleTransmission</type>
-    <joint name="right_wheel_hinge"/>
-    <actuator name="right_wheel_motor">
-      <mechanicalReduction>1</mechanicalReduction>
-    </actuator>
-  </transmission> -->
-  <!-- Gazebo ROS Control plugin -->
-  <!-- <gazebo>
-    <plugin name="gazebo_ros_control" filename="libgazebo_ros_control.so"/>
-  </gazebo> -->
 </robot>

Commit message: fixed wheel damping to lessen drift. added caster wheel.

File: ws/src/duckiebot_description/urdf/duckiebot.xacro (robot description, xacro)
@@ -111,4 +111,5 @@
     <origin xyz="0 0.07 0"/>
     <axis xyz="0 1 0"/>
+    <dynamics damping="0.1" friction="0.1"/>
   </joint>
   <joint type="continuous" name="right_wheel_hinge">
@@ -117,4 +118,5 @@
     <origin xyz="0 -0.07 0"/>
     <axis xyz="0 1 0"/>
+    <dynamics damping="0.1" friction="0.1"/>
   </joint>
   <!-- ======================= COMPUTER ======================= -->
@@ -217,8 +219,8 @@
       <plugin name="imu_plugin" filename="libgazebo_ros_imu_sensor.so">
         <ros>
-          <namespace>duckiebot</namespace>
+          <namespace></namespace>
         </ros>
-        <updateRateHZ>200</updateRateHZ>
-        <robotNamespace>duckiebot</robotNamespace>
+        <updateRateHZ>150</updateRateHZ>
+        <robotNamespace></robotNamespace>
         <topicName>imu/data</topicName>
         <frameName>imu_link</frameName>
@@ -227,4 +229,52 @@
     </sensor>
   </gazebo>
+  <!-- ======================= CASTER WHEEL ======================= -->
+  <link name="caster">
+    <inertial>
+      <mass value="${casterMass}"/>
+      <origin xyz="0 0 0"/>
+      <inertia ixx="1.0e-6" ixy="0" ixz="0"
+              iyy="1.0e-6" iyz="0"
+              izz="1.0e-6"/>
+    </inertial>
+    <visual>
+      <origin xyz="0 0 0" rpy="0 0 0"/>
+      <geometry>
+        <sphere radius="${casterRadius}"/>
+      </geometry>
+      <material name="black"/>
+    </visual>
+    <collision>
+      <origin xyz="0 0 0" rpy="0 0 0"/>
+      <geometry>
+        <sphere radius="${casterRadius}"/>
+      </geometry>
+      <surface>
+        <friction>
+          <ode>
+            <mu>0.0</mu>
+            <mu2>0.0</mu2>
+            <slip1>1.0</slip1>
+            <slip2>1.0</slip2>
+          </ode>
+        </friction>
+      </surface>
+    </collision>
+  </link>
+  <joint name="caster_joint" type="fixed">
+    <parent link="chassis"/>
+    <child link="caster"/>
+    <!-- Position caster at rear of robot, on ground level -->
+    <origin xyz="-${casterOffsetX} 0 ${-wheelRadius + casterRadius}" rpy="0 0 0"/>
+  </joint>
+  <gazebo reference="caster">
+    <material>Gazebo/Black</material>
+    <mu1>0.0</mu1>
+    <mu2>0.0</mu2>
+    <kp>100000.0</kp>
+    <kd>10.0</kd>
+    <minDepth>0.001</minDepth>
+    <maxVel>0.01</maxVel>
+  </gazebo>
   <!-- ======================= CAMERA ======================= -->
   <link name="camera">

Commit message: exp

File: ws/src/duckiebot_description/urdf/duckiebot.xacro (robot description, xacro)
@@ -177,42 +177,8 @@
       <imu>
         <angular_velocity>
-          <x>
-            <noise type="gaussian">
-              <mean>0.0</mean>
-              <stddev>0.0</stddev>
-            </noise>
-          </x>
-          <y>
-            <noise type="gaussian">
-              <mean>0.0</mean>
-              <stddev>0.0</stddev>
-            </noise>
-          </y>
-          <z>
-            <noise type="gaussian">
-              <mean>0.0</mean>
-              <stddev>0.0</stddev>
-            </noise>
-          </z>
+          <x>1</x><y>1</y><z>1</z>
         </angular_velocity>
         <linear_acceleration>
-          <x>
-            <noise type="gaussian">
-              <mean>0.0</mean>
-              <stddev>0.0</stddev>
-            </noise>
-          </x>
-          <y>
-            <noise type="gaussian">
-              <mean>0.0</mean>
-              <stddev>0.0</stddev>
-            </noise>
-          </y>
-          <z>
-            <noise type="gaussian">
-              <mean>0.0</mean>
-              <stddev>0.0</stddev>
-            </noise>
-          </z>
+          <x>1</x><y>1</y><z>1</z>
         </linear_acceleration>
       </imu>
@@ -225,56 +191,7 @@
         <topicName>imu/data</topicName>
         <frameName>imu_link</frameName>
-        <initialOrientationAsReference>false</initialOrientationAsReference>
       </plugin>
     </sensor>
   </gazebo>
-  <!-- ======================= CASTER WHEEL ======================= -->
-  <link name="caster">
-    <inertial>
-      <mass value="${casterMass}"/>
-      <origin xyz="0 0 0"/>
-      <inertia ixx="1.0e-6" ixy="0" ixz="0"
-              iyy="1.0e-6" iyz="0"
-              izz="1.0e-6"/>
-    </inertial>
-    <visual>
-      <origin xyz="0 0 0" rpy="0 0 0"/>
-      <geometry>
-        <sphere radius="${casterRadius}"/>
-      </geometry>
-      <material name="black"/>
-    </visual>
-    <collision>
-      <origin xyz="0 0 0" rpy="0 0 0"/>
-      <geometry>
-        <sphere radius="${casterRadius}"/>
-      </geometry>
-      <surface>
-        <friction>
-          <ode>
-            <mu>0.0</mu>
-            <mu2>0.0</mu2>
-            <slip1>1.0</slip1>
-            <slip2>1.0</slip2>
-          </ode>
-        </friction>
-      </surface>
-    </collision>
-  </link>
-  <joint name="caster_joint" type="fixed">
-    <parent link="chassis"/>
-    <child link="caster"/>
-    <!-- Position caster at rear of robot, on ground level -->
-    <origin xyz="-${casterOffsetX} 0 ${-wheelRadius + casterRadius}" rpy="0 0 0"/>
-  </joint>
-  <gazebo reference="caster">
-    <material>Gazebo/Black</material>
-    <mu1>0.0</mu1>
-    <mu2>0.0</mu2>
-    <kp>100000.0</kp>
-    <kd>10.0</kd>
-    <minDepth>0.001</minDepth>
-    <maxVel>0.01</maxVel>
-  </gazebo>
   <!-- ======================= CAMERA ======================= -->
   <link name="camera">
