Commit message: ros2 simulation environment, duckiebot does not appear in the wolrd for some reason

File: ws/src/duckiebot_description/urdf/duckiebot.xacro (robot description, xacro)
@@ -37,5 +37,6 @@
       <origin xyz="0 0 0"/>
       <geometry>
-        <mesh filename="package://duckiebot_description/meshes/duckiebotFrame.dae"/>
+        <!-- Original: <mesh filename="package://duckiebot_description/meshes/duckiebotFrame.dae"/> -->
+        <mesh filename="file://$(find duckiebot_description)/meshes/duckiebotFrame.dae" scale="0.001 0.001 0.001"/>
       </geometry>
       <material name="red"/>
@@ -44,5 +45,6 @@
       <origin xyz="0 0 0"/>
       <geometry>
-        <mesh filename="package://duckiebot_description/meshes/duckiebotFrame.dae"/>
+        <!-- Original: <mesh filename="package://duckiebot_description/meshes/duckiebotFrame.dae"/> -->
+        <mesh filename="file://$(find duckiebot_description)/meshes/duckiebotFrame.dae" scale="0.001 0.001 0.001"/>
       </geometry>
     </collision>
@@ -58,5 +60,6 @@
       <origin xyz="0 -0.07 0"/>
       <geometry>
-        <mesh filename="package://duckiebot_description/meshes/duckiebot_leftwheel.dae"/>
+        <!-- Original: <mesh filename="package://duckiebot_description/meshes/duckiebot_leftwheel.dae"/> -->
+        <mesh filename="file://$(find duckiebot_description)/meshes/duckiebot_leftwheel.dae" scale="0.001 0.001 0.001"/>
       </geometry>
       <material name="black"/>
@@ -65,5 +68,6 @@
       <origin xyz="0 -0.07 0"/>
       <geometry>
-        <mesh filename="package://duckiebot_description/meshes/duckiebot_leftwheel.dae"/>
+        <!-- Original: <mesh filename="package://duckiebot_description/meshes/duckiebot_leftwheel.dae"/> -->
+        <mesh filename="file://$(find duckiebot_description)/meshes/duckiebot_leftwheel.dae" scale="0.001 0.001 0.001"/>
       </geometry>
     </collision>
@@ -78,5 +82,6 @@
       <origin xyz="0 0.07 0"/>
       <geometry>
-        <mesh filename="package://duckiebot_description/meshes/duckiebot_rightwheel.dae"/>
+        <!-- Original: <mesh filename="package://duckiebot_description/meshes/duckiebot_rightwheel.dae"/> -->
+        <mesh filename="file://$(find duckiebot_description)/meshes/duckiebot_rightwheel.dae" scale="0.001 0.001 0.001"/>
       </geometry>
       <material name="black"/>
@@ -85,5 +90,6 @@
       <origin xyz="0 0.07 0"/>
       <geometry>
-        <mesh filename="package://duckiebot_description/meshes/duckiebot_rightwheel.dae"/>
+        <!-- Original: <mesh filename="package://duckiebot_description/meshes/duckiebot_rightwheel.dae"/> -->
+        <mesh filename="file://$(find duckiebot_description)/meshes/duckiebot_rightwheel.dae" scale="0.001 0.001 0.001"/>
       </geometry>
     </collision>
@@ -107,9 +113,11 @@
       <mass value="${compuMass}"/>
       <origin xyz="0 0 0"/>
-      <inertia ixx="1e-6" iyy="1e-6" izz="1e-6"/>
-    </inertial>
-    <visual>
-      <geometry>
-        <mesh filename="package://duckiebot_description/meshes/duckiebot_computer.dae"/>
+      <!-- Original: <inertia ixx="1e-6" iyy="1e-6" izz="1e-6"/> -->
+      <inertia ixx="1e-6" ixy="0" ixz="0" iyy="1e-6" iyz="0" izz="1e-6"/>
+    </inertial>
+    <visual>
+      <geometry>
+        <!-- Original: <mesh filename="package://duckiebot_description/meshes/duckiebot_computer.dae"/> -->
+        <mesh filename="file://$(find duckiebot_description)/meshes/duckiebot_computer.dae" scale="0.001 0.001 0.001"/>
       </geometry>
       <material name="blue"/>
@@ -117,5 +125,6 @@
     <collision>
       <geometry>
-        <mesh filename="package://duckiebot_description/meshes/duckiebot_computer.dae"/>
+        <!-- Original: <mesh filename="package://duckiebot_description/meshes/duckiebot_computer.dae"/> -->
+        <mesh filename="file://$(find duckiebot_description)/meshes/duckiebot_computer.dae" scale="0.001 0.001 0.001"/>
       </geometry>
     </collision>
@@ -130,5 +139,6 @@
       <mass value="0.01"/>
       <origin xyz="0 0 0"/>
-      <inertia ixx="1e-6" iyy="1e-6" izz="1e-6"/>
+      <!-- Original: <inertia ixx="1e-6" iyy="1e-6" izz="1e-6"/> -->
+      <inertia ixx="1e-6" ixy="0" ixz="0" iyy="1e-6" iyz="0" izz="1e-6"/>
     </inertial>
     <visual>
@@ -152,5 +162,5 @@
     <sensor type="imu" name="imu_sensor">
       <always_on>true</always_on>
-      <updateRateHZ>50</updateRateHZ>
+      <update_rate>50</update_rate>
       <imu>
         <angular_velocity>
@@ -197,14 +207,9 @@
       <plugin name="imu_plugin" filename="libgazebo_ros_imu_sensor.so">
         <ros>
-          <namespace>duckiebot</namespace>
+          <namespace>/duckiebot</namespace>
+          <remapping>~/out:=imu/data</remapping>
         </ros>
-        <robotNamespace>duckiebot</robotNamespace>
-        <topicName>imu/data</topicName>
-        <frameName>imu_link</frameName>
-        <updateRateHZ>50</updateRateHZ>
-        <gaussianNoise>0.0</gaussianNoise>
-        <xyzOffset>0 0 0</xyzOffset>
-        <rpyOffset>0 0 0</rpyOffset>
-        <initialOrientationAsReference>false</initialOrientationAsReference>
+        <frame_name>imu_link</frame_name>
+        <initial_orientation_as_reference>false</initial_orientation_as_reference>
       </plugin>
     </sensor>
@@ -215,10 +220,12 @@
       <mass value="${cameraMass}"/>
       <origin xyz="0 0 0"/>
-      <inertia ixx="1e-6" iyy="1e-6" izz="1e-6"/>
+      <!-- Original: <inertia ixx="1e-6" iyy="1e-6" izz="1e-6"/> -->
+      <inertia ixx="1e-6" ixy="0" ixz="0" iyy="1e-6" iyz="0" izz="1e-6"/>
     </inertial>
     <visual>
       <origin xyz="-0.05 0 -0.055" rpy="0 -0.1 0"/>
       <geometry>
-        <mesh filename="package://duckiebot_description/meshes/duckiebot_camera.dae"/>
+        <!-- Original: <mesh filename="package://duckiebot_description/meshes/duckiebot_camera.dae"/> -->
+        <mesh filename="file://$(find duckiebot_description)/meshes/duckiebot_camera.dae" scale="0.001 0.001 0.001"/>
       </geometry>
       <material name="black"/>
@@ -227,5 +234,6 @@
       <origin xyz="-0.05 0 -0.055" rpy="0 -0.1 0"/>
       <geometry>
-        <mesh filename="package://duckiebot_description/meshes/duckiebot_camera.dae"/>
+        <!-- Original: <mesh filename="package://duckiebot_description/meshes/duckiebot_camera.dae"/> -->
+        <mesh filename="file://$(find duckiebot_description)/meshes/duckiebot_camera.dae" scale="0.001 0.001 0.001"/>
       </geometry>
     </collision>
